Commit message: Adding RFID URDF comp
-Also reinitializing bringup to launch rfid_node

File: turtlebot3_description/urdf/turtlebot3_burger.urdf (robot description, URDF)
Before this commit: robot turtlebot3_burger, 7 links, 6 joints
Links:
- added link rfid_base_link; collision box size=0.140 0.140 0.143; visual mesh filename=package://turtlebot3_description/meshes/bases/rfid_base.stl scale=0.001 0.001 0.001
Joints:
- added joint rfid_base_joint: type fixed, parent base_link, child rfid_base_link, origin xyz=0.0 0.08 0.023 rpy=0 0 0, axis 0 0 1

Commit message: Update turtlebot3_burger.urdf

File: turtlebot3_description/urdf/turtlebot3_burger.urdf (robot description, URDF)
Before this commit: robot turtlebot3_burger, 8 links, 7 joints
Links:
- link rfid_base_link: geometry collision box size=0.140 0.140 0.143; visual mesh filename=package://turtlebot3_description/meshes/bases/rfid_base.stl scale=1 1 1
Joints:
- joint rfid_base_joint: axis 0 0 1 -> (none); origin xyz=0.0 0.08 0.023 rpy=0 0 0 -> xyz=-0.14 0.0 0.0 rpy=0 0 0

Commit message: tweaking urdf location

File: turtlebot3_description/urdf/turtlebot3_burger.urdf (robot description, URDF)
Before this commit: robot turtlebot3_burger, 8 links, 7 joints
Joints:
- joint rfid_base_joint: origin xyz=-0.14 0.0 0.0 rpy=0 0 0 -> xyz=-0.14 0.0 0.2 rpy=0 0 0

Commit message: Update turtlebot3_burger.urdf

File: turtlebot3_description/urdf/turtlebot3_burger.urdf (robot description, URDF)
Before this commit: robot turtlebot3_burger, 8 links, 7 joints
Links:
- link rfid_base_link: geometry collision box size=0.140 0.140 0.143; visual mesh filename=package://turtlebot3_description/meshes/bases/rfid_base.stl scale=0.1 0.1 0.1

Commit message: Update turtlebot3_burger.urdf

File: turtlebot3_description/urdf/turtlebot3_burger.urdf (robot description, URDF)
Before this commit: robot turtlebot3_burger, 8 links, 7 joints
Links:
- link rfid_base_link: geometry collision box size=0.140 0.140 0.143; visual mesh filename=package://turtlebot3_description/meshes/bases/rfid_base.stl scale=0.001 0.001 0.001

Commit message: Update turtlebot3_burger.urdf

File: turtlebot3_description/urdf/turtlebot3_burger.urdf (robot description, URDF)
Before this commit: robot turtlebot3_burger, 8 links, 7 joints
Joints:
- joint rfid_base_joint: origin xyz=-0.14 0.0 0.2 rpy=0 0 0 -> xyz=-0.11 0.0 0.075 rpy=0 0 0

Commit message: Update turtlebot3_burger.urdf

File: turtlebot3_description/urdf/turtlebot3_burger.urdf (robot description, URDF)
Before this commit: robot turtlebot3_burger, 8 links, 7 joints
Joints:
- joint rfid_base_joint: origin xyz=-0.11 0.0 0.075 rpy=0 0 0 -> xyz=-0.08 0.0 0.1 rpy=0 0 0

Commit message: Update turtlebot3_burger.urdf

File: turtlebot3_description/urdf/turtlebot3_burger.urdf (robot description, URDF)
Before this commit: robot turtlebot3_burger, 8 links, 7 joints
Joints:
- joint rfid_base_joint: origin xyz=-0.08 0.0 0.1 rpy=0 0 0 -> xyz=-0.08 0.1 0.085 rpy=0 0 0

Commit message: Update turtlebot3_burger.urdf

File: turtlebot3_description/urdf/turtlebot3_burger.urdf (robot description, URDF)
Before this commit: robot turtlebot3_burger, 8 links, 7 joints
Joints:
- joint rfid_base_joint: origin xyz=-0.08 0.1 0.085 rpy=0 0 0 -> xyz=-0.085 0.01 0.09 rpy=0 0 0

Commit message: Update turtlebot3_burger.urdf

File: turtlebot3_description/urdf/turtlebot3_burger.urdf (robot description, URDF)
Before this commit: robot turtlebot3_burger, 8 links, 7 joints
Joints:
- joint rfid_base_joint: origin xyz=-0.085 0.01 0.09 rpy=0 0 0 -> xyz=-0.085 0.02 0.085 rpy=0 0 0

Commit message: Update turtlebot3_burger.urdf

File: turtlebot3_description/urdf/turtlebot3_burger.urdf (robot description, URDF)
Before this commit: robot turtlebot3_burger, 8 links, 7 joints
Joints:
- joint rfid_base_joint: origin xyz=-0.085 0.02 0.085 rpy=0 0 0 -> xyz=-0.085 0.015 0.0875 rpy=0 0 0

Commit message: Update turtlebot3_burger.urdf

File: turtlebot3_description/urdf/turtlebot3_burger.urdf (robot description, URDF)
Before this commit: robot turtlebot3_burger, 8 links, 7 joints
Joints:
- joint rfid_base_joint: origin xyz=-0.085 0.015 0.0875 rpy=0 0 0 -> xyz=-0.0825 0.015 0.085 rpy=0 0 0

Commit message: Update turtlebot3_burger.urdf

File: turtlebot3_description/urdf/turtlebot3_burger.urdf (robot description, URDF)
Before this commit: robot turtlebot3_burger, 8 links, 7 joints
Joints:
- joint rfid_base_joint: origin xyz=-0.0825 0.015 0.085 rpy=0 0 0 -> xyz=-0.01 0.0125 0.0825 rpy=0 0 0

Commit message: Update turtlebot3_burger.urdf

File: turtlebot3_description/urdf/turtlebot3_burger.urdf (robot description, URDF)
Before this commit: robot turtlebot3_burger, 8 links, 7 joints
Joints:
- joint rfid_base_joint: origin xyz=-0.01 0.0125 0.0825 rpy=0 0 0 -> xyz=-0.1 0.0125 0.0825 rpy=0 0 0

Commit message: Update turtlebot3_burger.urdf

File: turtlebot3_description/urdf/turtlebot3_burger.urdf (robot description, URDF)
Before this commit: robot turtlebot3_burger, 8 links, 7 joints
Joints:
- joint rfid_base_joint: origin xyz=-0.1 0.0125 0.0825 rpy=0 0 0 -> xyz=-0.1 0.0125 0.084 rpy=0 0 0

Commit message: Update turtlebot3_burger.urdf

File: turtlebot3_description/urdf/turtlebot3_burger.urdf (robot description, URDF)
Before this commit: robot turtlebot3_burger, 8 links, 7 joints
Joints:
- joint rfid_base_joint: origin xyz=-0.1 0.0125 0.084 rpy=0 0 0 -> xyz=-0.825 0.0125 0.0845 rpy=0 0 0

Commit message: Update turtlebot3_burger.urdf

File: turtlebot3_description/urdf/turtlebot3_burger.urdf (robot description, URDF)
Before this commit: robot turtlebot3_burger, 8 links, 7 joints
Joints:
- joint rfid_base_joint: origin xyz=-0.825 0.0125 0.0845 rpy=0 0 0 -> xyz=-0.1 0.0125 0.085 rpy=0 0 0

Commit message: Update turtlebot3_burger.urdf

File: turtlebot3_description/urdf/turtlebot3_burger.urdf (robot description, URDF)
Before this commit: robot turtlebot3_burger, 8 links, 7 joints
Joints:
- joint rfid_base_joint: origin xyz=-0.1 0.0125 0.085 rpy=0 0 0 -> xyz=-0.9 0.0125 0.086 rpy=0 0 0

Commit message: Update turtlebot3_burger.urdf

File: turtlebot3_description/urdf/turtlebot3_burger.urdf (robot description, URDF)
Before this commit: robot turtlebot3_burger, 8 links, 7 joints
Joints:
- joint rfid_base_joint: origin xyz=-0.9 0.0125 0.086 rpy=0 0 0 -> xyz=-0.9 0.0125 0.087 rpy=0 0 0

Commit message: Update turtlebot3_burger.urdf

File: turtlebot3_description/urdf/turtlebot3_burger.urdf (robot description, URDF)
Before this commit: robot turtlebot3_burger, 8 links, 7 joints
Joints:
- joint rfid_base_joint: origin xyz=-0.9 0.0125 0.087 rpy=0 0 0 -> xyz=-0.09 0.0125 0.087 rpy=0 0 0

Commit message: Update turtlebot3_burger.urdf

File: turtlebot3_description/urdf/turtlebot3_burger.urdf (robot description, URDF)
Before this commit: robot turtlebot3_burger, 8 links, 7 joints
Joints:
- joint rfid_base_joint: origin xyz=-0.09 0.0125 0.087 rpy=0 0 0 -> xyz=-0.088 0.0125 0.087 rpy=0 0 0

Commit message: Update turtlebot3_burger.urdf

File: turtlebot3_description/urdf/turtlebot3_burger.urdf (robot description, URDF)
Before this commit: robot turtlebot3_burger, 8 links, 7 joints
Joints:
- joint rfid_base_joint: origin xyz=-0.088 0.0125 0.087 rpy=0 0 0 -> xyz=-0.0875 0.0125 0.087 rpy=0 0 0

Commit message: Update turtlebot3_burger.urdf

File: turtlebot3_description/urdf/turtlebot3_burger.urdf (robot description, URDF)
Before this commit: robot turtlebot3_burger, 8 links, 7 joints
Joints:
- joint rfid_base_joint: origin xyz=-0.0875 0.0125 0.087 rpy=0 0 0 -> xyz=-0.087 0.0125 0.087 rpy=0 0 0

Commit message: Update turtlebot3_burger.urdf

File: turtlebot3_description/urdf/turtlebot3_burger.urdf (robot description, URDF)
Before this commit: robot turtlebot3_burger, 8 links, 7 joints
Joints:
- joint rfid_base_joint: origin xyz=-0.087 0.0125 0.087 rpy=0 0 0 -> xyz=-0.08675 0.0125 0.087 rpy=0 0 0

Commit message: Update turtlebot3_burger.urdf

File: turtlebot3_description/urdf/turtlebot3_burger.urdf (robot description, URDF)
Before this commit: robot turtlebot3_burger, 8 links, 7 joints
Joints:
- joint rfid_base_joint: origin xyz=-0.08675 0.0125 0.087 rpy=0 0 0 -> xyz=-0.086 0.0125 0.087 rpy=0 0 0

Commit message: Update turtlebot3_burger.urdf

File: turtlebot3_description/urdf/turtlebot3_burger.urdf (robot description, URDF)
Before this commit: robot turtlebot3_burger, 8 links, 7 joints
Joints:
- joint rfid_base_joint: origin xyz=-0.086 0.0125 0.087 rpy=0 0 0 -> xyz=-0.0855 0.0125 0.087 rpy=0 0 0

Commit message: Update turtlebot3_burger.urdf

File: turtlebot3_description/urdf/turtlebot3_burger.urdf (robot description, URDF)
Before this commit: robot turtlebot3_burger, 8 links, 7 joints
Joints:
- joint rfid_base_joint: origin xyz=-0.0855 0.0125 0.087 rpy=0 0 0 -> xyz=-0.085 0.0125 0.087 rpy=0 0 0

Commit message: Update turtlebot3_burger.urdf

File: turtlebot3_description/urdf/turtlebot3_burger.urdf (robot description, URDF)
Before this commit: robot turtlebot3_burger, 8 links, 7 joints
Links:
- added link rfid_sensor_link; visual box size=0.005 0.05 0.08
Joints:
- added joint rfid_sensor_joint: type fixed, parent rfid_base_link, child rfid_sensor_link, origin xyz=-0.1 0.1 0.1 rpy=0 0 1.57079632679

Commit message: Update turtlebot3_burger.urdf

File: turtlebot3_description/urdf/turtlebot3_burger.urdf (robot description, URDF)
Before this commit: robot turtlebot3_burger, 9 links, 8 joints
Joints:
- joint rfid_sensor_joint: origin xyz=-0.1 0.1 0.1 rpy=0 0 1.57079632679 -> xyz=-0.5 0.05 0.05 rpy=0 0 1.57079632679

Commit message: Update turtlebot3_burger.urdf

File: turtlebot3_description/urdf/turtlebot3_burger.urdf (robot description, URDF)
Before this commit: robot turtlebot3_burger, 9 links, 8 joints
Joints:
- joint rfid_sensor_joint: origin xyz=-0.5 0.05 0.05 rpy=0 0 1.57079632679 -> xyz=-0.05 0.05 0.05 rpy=0 0 1.57079632679

Commit message: Update turtlebot3_burger.urdf

File: turtlebot3_description/urdf/turtlebot3_burger.urdf (robot description, URDF)
Before this commit: robot turtlebot3_burger, 9 links, 8 joints
Links:
- added link rfid_sensor_measure; visual box size=0.005 0.05 0.08
- link rfid_sensor_link: geometry visual box size=0.005 0.04 0.08
Joints:
- joint rfid_sensor_joint: child rfid_sensor_link -> rfid_sensor_measure; origin xyz=-0.05 0.05 0.05 rpy=0 0 1.57079632679 -> xyz=0 0.0 0.05 rpy=0 0 0; parent rfid_base_link -> rfid_sensor_link

Commit message: Update turtlebot3_burger.urdf

File: turtlebot3_description/urdf/turtlebot3_burger.urdf (robot description, URDF)
Before this commit: robot turtlebot3_burger, 10 links, 8 joints
Links:
- removed link rfid_sensor_measure
- link rfid_sensor_link: geometry visual box size=0.005 0.05 0.08
Joints:
- joint rfid_sensor_joint: child rfid_sensor_measure -> rfid_sensor_link; origin xyz=0 0.0 0.05 rpy=0 0 0 -> xyz=-0.04 0.05 0.05 rpy=0 0 1.57079632679; parent rfid_sensor_link -> rfid_base_link

Commit message: Update turtlebot3_burger.urdf

File: turtlebot3_description/urdf/turtlebot3_burger.urdf (robot description, URDF)
Before this commit: robot turtlebot3_burger, 9 links, 8 joints
Joints:
- joint rfid_sensor_joint: origin xyz=-0.04 0.05 0.05 rpy=0 0 1.57079632679 -> xyz=-0.0425 0.05 0 rpy=0 0 1.57079632679

Commit message: Update turtlebot3_burger.urdf

File: turtlebot3_description/urdf/turtlebot3_burger.urdf (robot description, URDF)
Before this commit: robot turtlebot3_burger, 9 links, 8 joints
Links:
- link rfid_sensor_link: geometry visual box size=0.001 0.05 0.08
Joints:
- joint rfid_sensor_joint: origin xyz=-0.0425 0.05 0 rpy=0 0 1.57079632679 -> xyz=-0.0425 0.05 -0.05 rpy=0 0 1.57079632679

Commit message: Update turtlebot3_burger.urdf

File: turtlebot3_description/urdf/turtlebot3_burger.urdf (robot description, URDF)
Before this commit: robot turtlebot3_burger, 9 links, 8 joints
Joints:
- joint rfid_sensor_joint: origin xyz=-0.0425 0.05 -0.05 rpy=0 0 1.57079632679 -> xyz=-0.0425 0.02 -0.025 rpy=0 0 1.57079632679

Commit message: Update turtlebot3_burger.urdf

File: turtlebot3_description/urdf/turtlebot3_burger.urdf (robot description, URDF)
Before this commit: robot turtlebot3_burger, 9 links, 8 joints
Joints:
- joint rfid_sensor_joint: origin xyz=-0.0425 0.02 -0.025 rpy=0 0 1.57079632679 -> xyz=-0.0425 0.035 -0.015 rpy=0 0 1.57079632679

Commit message: Update turtlebot3_burger.urdf

File: turtlebot3_description/urdf/turtlebot3_burger.urdf (robot description, URDF)
Before this commit: robot turtlebot3_burger, 9 links, 8 joints
Joints:
- joint rfid_sensor_joint: origin xyz=-0.0425 0.035 -0.015 rpy=0 0 1.57079632679 -> xyz=-0.0425 0.05 0 rpy=0 0 1.57079632679

Commit message: Update turtlebot3_burger.urdf

File: turtlebot3_description/urdf/turtlebot3_burger.urdf (robot description, URDF)
Before this commit: robot turtlebot3_burger, 9 links, 8 joints
Joints:
- joint rfid_sensor_joint: origin xyz=-0.0425 0.05 0 rpy=0 0 1.57079632679 -> xyz=-0.0425 0.045 .005 rpy=0 0 1.57079632679

Commit message: Update turtlebot3_burger.urdf

File: turtlebot3_description/urdf/turtlebot3_burger.urdf (robot description, URDF)
Before this commit: robot turtlebot3_burger, 9 links, 8 joints
Joints:
- joint rfid_sensor_joint: origin xyz=-0.0425 0.045 .005 rpy=0 0 1.57079632679 -> xyz=-0.0425 0.045 .01 rpy=0 0 1.57079632679

Commit message: Update turtlebot3_burger.urdf

File: turtlebot3_description/urdf/turtlebot3_burger.urdf (robot description, URDF)
Before this commit: robot turtlebot3_burger, 9 links, 8 joints
Joints:
- joint rfid_sensor_joint: origin xyz=-0.0425 0.045 .01 rpy=0 0 1.57079632679 -> xyz=-0.0425 0.045 .012 rpy=0 0 1.57079632679

Commit message: Update turtlebot3_burger.urdf

File: turtlebot3_description/urdf/turtlebot3_burger.urdf (robot description, URDF)
Before this commit: robot turtlebot3_burger, 9 links, 8 joints
Joints:
- joint rfid_sensor_joint: origin xyz=-0.0425 0.045 .012 rpy=0 0 1.57079632679 -> xyz=-0.0425 0.045 .013 rpy=0 0 1.57079632679

Commit message: Update turtlebot3_burger.urdf

File: turtlebot3_description/urdf/turtlebot3_burger.urdf (robot description, URDF)
Before this commit: robot turtlebot3_burger, 9 links, 8 joints
Joints:
- joint rfid_sensor_joint: origin xyz=-0.0425 0.045 .013 rpy=0 0 1.57079632679 -> xyz=-0.0425 0.045 .014 rpy=0 0 1.57079632679

Commit message: Update turtlebot3_burger.urdf

File: turtlebot3_description/urdf/turtlebot3_burger.urdf (robot description, URDF)
Before this commit: robot turtlebot3_burger, 9 links, 8 joints
Joints:
- joint rfid_sensor_joint: origin xyz=-0.0425 0.045 .014 rpy=0 0 1.57079632679 -> xyz=-0.0425 0.045 .02 rpy=0 0 1.57079632679

Commit message: Update turtlebot3_burger.urdf

File: turtlebot3_description/urdf/turtlebot3_burger.urdf (robot description, URDF)
Before this commit: robot turtlebot3_burger, 9 links, 8 joints
Joints:
- joint rfid_sensor_joint: origin xyz=-0.0425 0.045 .02 rpy=0 0 1.57079632679 -> xyz=-0.0425 0.045 .04 rpy=0 0 1.57079632679

Commit message: Update turtlebot3_burger.urdf

File: turtlebot3_description/urdf/turtlebot3_burger.urdf (robot description, URDF)
Before this commit: robot turtlebot3_burger, 9 links, 8 joints
Joints:
- joint rfid_sensor_joint: origin xyz=-0.0425 0.045 .04 rpy=0 0 1.57079632679 -> xyz=-0.0425 0.045 .035 rpy=0 0 1.57079632679
